File: Documents/Eagle CAD/piSchoolBell-12pinLCD.sch (EAGLE design)
At the start: 17 parts, among them J1 455-1750-1-ND, X1 RASPI_BOARD_B+#_H

Commit message: Routed PCB
Other:
- moved on the sheet: SV2
Changed lines of the file:
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@@
 <attribute name="VALUE" x="250.19" y="64.77" size="1.778" layer="96" rot="R180"/>
 </instance>
-<instance part="SV2" gate="G$1" x="200.66" y="116.84" smashed="yes">
-<attribute name="NAME" x="196.85" y="122.682" size="1.778" layer="95"/>
+<instance part="SV2" gate="G$1" x="200.66" y="104.14" smashed="yes">
+<attribute name="NAME" x="196.85" y="109.982" size="1.778" layer="95"/>
 </instance>
 <instance part="SV3" gate="G$1" x="170.18" y="243.84" smashed="yes" rot="R180">
@@
 <wire x1="264.16" y1="142.24" x2="236.22" y2="142.24" width="0.1524" layer="91"/>
 <pinref part="SV2" gate="G$1" pin="RS"/>
-<wire x1="208.28" y1="99.06" x2="236.22" y2="99.06" width="0.1524" layer="91"/>
+<wire x1="210.82" y1="99.06" x2="236.22" y2="99.06" width="0.1524" layer="91"/>
 <wire x1="236.22" y1="99.06" x2="236.22" y2="142.24" width="0.1524" layer="91"/>
 </segment>
@@
 <wire x1="233.68" y1="139.7" x2="264.16" y2="139.7" width="0.1524" layer="91"/>
 <pinref part="SV2" gate="G$1" pin="E"/>
-<wire x1="208.28" y1="104.14" x2="233.68" y2="104.14" width="0.1524" layer="91"/>
+<wire x1="210.82" y1="104.14" x2="233.68" y2="104.14" width="0.1524" layer="91"/>
 <wire x1="233.68" y1="104.14" x2="233.68" y2="139.7" width="0.1524" layer="91"/>
 </segment>
@@
 <wire x1="231.14" y1="157.48" x2="264.16" y2="157.48" width="0.1524" layer="91"/>
 <pinref part="SV2" gate="G$1" pin="D4"/>
-<wire x1="208.28" y1="106.68" x2="231.14" y2="106.68" width="0.1524" layer="91"/>
+<wire x1="210.82" y1="106.68" x2="231.14" y2="106.68" width="0.1524" layer="91"/>
 </segment>
 </net>
@@
 <wire x1="228.6" y1="152.4" x2="264.16" y2="152.4" width="0.1524" layer="91"/>
 <pinref part="SV2" gate="G$1" pin="D5"/>
-<wire x1="208.28" y1="109.22" x2="228.6" y2="109.22" width="0.1524" layer="91"/>
+<wire x1="210.82" y1="109.22" x2="228.6" y2="109.22" width="0.1524" layer="91"/>
 </segment>
 </net>
@@
 <wire x1="226.06" y1="149.86" x2="226.06" y2="111.76" width="0.1524" layer="91"/>
 <pinref part="SV2" gate="G$1" pin="D6"/>
-<wire x1="208.28" y1="111.76" x2="226.06" y2="111.76" width="0.1524" layer="91"/>
+<wire x1="210.82" y1="111.76" x2="226.06" y2="111.76" width="0.1524" layer="91"/>
 </segment>
 </net>
@@
 <wire x1="223.52" y1="144.78" x2="223.52" y2="114.3" width="0.1524" layer="91"/>
 <pinref part="SV2" gate="G$1" pin="D7"/>
-<wire x1="208.28" y1="114.3" x2="223.52" y2="114.3" width="0.1524" layer="91"/>
+<wire x1="210.82" y1="114.3" x2="223.52" y2="114.3" width="0.1524" layer="91"/>
 </segment>
 </net>
@@
 <wire x1="220.98" y1="203.2" x2="284.48" y2="203.2" width="0.1524" layer="91"/>
 <pinref part="SV2" gate="G$1" pin="LED+"/>
-<wire x1="220.98" y1="116.84" x2="208.28" y2="116.84" width="0.1524" layer="91"/>
+<wire x1="220.98" y1="116.84" x2="210.82" y2="116.84" width="0.1524" layer="91"/>
 <pinref part="SV3" gate="G$1" pin="VCC#2"/>
 <wire x1="284.48" y1="203.2" x2="284.48" y2="241.3" width="0.1524" layer="91"/>
@@
 <pinref part="R10" gate="1" pin="E"/>
 <pinref part="SV2" gate="G$1" pin="VCC"/>
-<wire x1="208.28" y1="93.98" x2="238.76" y2="93.98" width="0.1524" layer="91"/>
+<wire x1="210.82" y1="93.98" x2="238.76" y2="93.98" width="0.1524" layer="91"/>
 <junction x="238.76" y="93.98"/>
 </segment>
@@
 <pinref part="R10" gate="1" pin="A"/>
 <pinref part="SV2" gate="G$1" pin="LED-"/>
-<wire x1="208.28" y1="119.38" x2="307.34" y2="119.38" width="0.1524" layer="91"/>
+<wire x1="210.82" y1="119.38" x2="307.34" y2="119.38" width="0.1524" layer="91"/>
 <junction x="307.34" y="119.38"/>
 <pinref part="SV2" gate="G$1" pin="R/W"/>
-<wire x1="208.28" y1="101.6" x2="307.34" y2="101.6" width="0.1524" layer="91"/>
+<wire x1="210.82" y1="101.6" x2="307.34" y2="101.6" width="0.1524" layer="91"/>
 <junction x="307.34" y="101.6"/>
 <pinref part="SV2" gate="G$1" pin="GND"/>
-<wire x1="208.28" y1="91.44" x2="307.34" y2="91.44" width="0.1524" layer="91"/>
+<wire x1="210.82" y1="91.44" x2="307.34" y2="91.44" width="0.1524" layer="91"/>
 <junction x="307.34" y="91.44"/>
 <pinref part="SV3" gate="G$1" pin="GND#2"/>
@@
 <pinref part="SV2" gate="G$1" pin="VO"/>
 <wire x1="246.38" y1="73.66" x2="246.38" y2="96.52" width="0.1524" layer="91"/>
-<wire x1="246.38" y1="96.52" x2="208.28" y2="96.52" width="0.1524" layer="91"/>
-</segment>
-</net>
+<wire x1="246.38" y1="96.52" x2="210.82" y2="96.52" width="0.1524" layer="91"/>
+</segment>
+</net>

Commit message: Coppper pour on pdfs
Connections:
- net N$27 renamed GND
Changed lines of the file:
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@@
 </segment>
 </net>
-<net name="N$27" class="0">
+<net name="GND" class="0">
 <segment>
 <pinref part="X1" gate="G$1" pin="GND_A"/>
