File: KiCad/piSchoolBell/piSchoolBell.kicad_pcb (KiCad board)
At the start: 2 copper layers, 99.7 x 71.1 mm, 16 parts, among them J3 Raspberry_Pi_2_3_all_pin_orde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, J4 3-pin_KY-019_relay_header, U1 LCD_HD44780, U2 5-pin_4_buttons_+_common, U3 DS3231_RTC_module

Commit message: minor schematic change
Parts:
- J4: value 3-pin_KY-019_relay_header -> Bell relay
