File: KiCad/piSchoolBell/piSchoolBell.kicad_sch (KiCad schematic)
At the start: 16 parts, among them U1 LCD_HD44780, U2 5-pin_4_buttons_+_common, U3 DS3231_RTC_module

Commit message: minor schematic change
Parts:
- D1: value (none) -> LED; footprint (none) -> My_Misc:LED_D5.0mm_larger_pads
- J3: value (none) -> Raspberry_Pi_2_3_all_pin_ordered
- J4: value (none) -> Bell relay
- R1, R2, R3, R4: value (none) -> 300R; footprint (none) -> My_Misc:R_Axial_DIN0207_L6.3mm_D2.5mm_P10.16mm_Horizontal_larger_pads
- R5, R6, R7, R8: value (none) -> 10k; footprint (none) -> My_Misc:R_Axial_DIN0207_L6.3mm_D2.5mm_P10.16mm_Horizontal_larger_pads
- R9: value (none) -> 220R; footprint (none) -> My_Misc:R_Axial_DIN0207_L6.3mm_D2.5mm_P10.16mm_Horizontal_larger_pads
Changed lines of the file:
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@@
     (in_bom yes) (on_board yes)
     (property "Reference" "J3" (id 0) (at 148.59 61.7982 0))
-    (property "Value" "" (id 1) (at 148.59 64.1096 0))
+    (property "Value" "Raspberry_Pi_2_3_all_pin_ordered" (id 1) (at 148.59 64.1096 0))
     (property "Footprint" "My_RaspberryPi:RaspberryPi_3b+_Hat_large" (id 2) (at 148.59 96.52 0)
       (effects (font (size 1.27 1.27)) hide)
@@
     (in_bom yes) (on_board yes)
     (property "Reference" "D1" (id 0) (at 250.3678 68.453 0))
-    (property "Value" "" (id 1) (at 250.3678 70.7644 0))
-    (property "Footprint" "" (id 2) (at 250.19 74.93 0)
+    (property "Value" "LED" (id 1) (at 250.3678 70.7644 0))
+    (property "Footprint" "My_Misc:LED_D5.0mm_larger_pads" (id 2) (at 250.19 74.93 0)
       (effects (font (size 1.27 1.27)) hide)
     )
@@
     (in_bom yes) (on_board yes)
     (property "Reference" "R9" (id 0) (at 250.19 59.5122 90))
-    (property "Value" "" (id 1) (at 250.19 61.8236 90))
-    (property "Footprint" "" (id 2) (at 250.19 62.992 90)
+    (property "Value" "220R" (id 1) (at 250.19 61.8236 90))
+    (property "Footprint" "My_Misc:R_Axial_DIN0207_L6.3mm_D2.5mm_P10.16mm_Horizontal_larger_pads" (id 2) (at 250.19 62.992 90)
       (effects (font (size 1.27 1.27)) hide)
     )
@@
       (effects (font (size 1.27 1.27)) (justify left))
     )
-    (property "Value" "" (id 1) (at 251.46 88.9 0)
-      (effects (font (size 1.27 1.27)) hide)
-    )
+    (property "Value" "Bell relay" (id 1) (at 251.46 88.9 0))
     (property "Footprint" "My_Headers:3-pin JST KY-019 relay" (id 2) (at 251.46 91.44 0)
       (effects (font (size 1.27 1.27)) hide)
@@
     (in_bom yes) (on_board yes)
     (property "Reference" "R1" (id 0) (at 200.66 88.7222 90))
-    (property "Value" "" (id 1) (at 200.66 91.0336 90))
-    (property "Footprint" "" (id 2) (at 200.66 92.202 90)
+    (property "Value" "300R" (id 1) (at 200.66 91.0336 90))
+    (property "Footprint" "My_Misc:R_Axial_DIN0207_L6.3mm_D2.5mm_P10.16mm_Horizontal_larger_pads" (id 2) (at 200.66 92.202 90)
       (effects (font (size 1.27 1.27)) hide)
     )
@@
     (in_bom yes) (on_board yes)
     (property "Reference" "R2" (id 0) (at 200.66 100.1522 90))
-    (property "Value" "" (id 1) (at 200.66 102.4636 90))
-    (property "Footprint" "" (id 2) (at 200.66 103.632 90)
+    (property "Value" "300R" (id 1) (at 200.66 102.4636 90))
+    (property "Footprint" "My_Misc:R_Axial_DIN0207_L6.3mm_D2.5mm_P10.16mm_Horizontal_larger_pads" (id 2) (at 200.66 103.632 90)
       (effects (font (size 1.27 1.27)) hide)
     )
@@
     (in_bom yes) (on_board yes)
     (property "Reference" "R3" (id 0) (at 200.66 110.3122 90))
-    (property "Value" "" (id 1) (at 200.66 112.6236 90))
-    (property "Footprint" "" (id 2) (at 200.66 113.792 90)
+    (property "Value" "300R" (id 1) (at 200.66 112.6236 90))
+    (property "Footprint" "My_Misc:R_Axial_DIN0207_L6.3mm_D2.5mm_P10.16mm_Horizontal_larger_pads" (id 2) (at 200.66 113.792 90)
       (effects (font (size 1.27 1.27)) hide)
     )
@@
     (in_bom yes) (on_board yes)
     (property "Reference" "R4" (id 0) (at 200.66 120.4722 90))
-    (property "Value" "" (id 1) (at 200.66 122.7836 90))
-    (property "Footprint" "" (id 2) (at 200.66 123.952 90)
+    (property "Value" "300R" (id 1) (at 200.66 122.7836 90))
+    (property "Footprint" "My_Misc:R_Axial_DIN0207_L6.3mm_D2.5mm_P10.16mm_Horizontal_larger_pads" (id 2) (at 200.66 123.952 90)
       (effects (font (size 1.27 1.27)) hide)
     )
@@
     (in_bom yes) (on_board yes)
     (property "Reference" "R5" (id 0) (at 217.17 86.1822 90))
-    (property "Value" "" (id 1) (at 217.17 88.4936 90))
-    (property "Footprint" "" (id 2) (at 217.17 89.662 90)
+    (property "Value" "10k" (id 1) (at 217.17 88.4936 90))
+    (property "Footprint" "My_Misc:R_Axial_DIN0207_L6.3mm_D2.5mm_P10.16mm_Horizontal_larger_pads" (id 2) (at 217.17 89.662 90)
       (effects (font (size 1.27 1.27)) hide)
     )
@@
     (in_bom yes) (on_board yes)
     (property "Reference" "R6" (id 0) (at 217.17 97.6122 90))
-    (property "Value" "" (id 1) (at 217.17 99.9236 90))
-    (property "Footprint" "" (id 2) (at 217.17 101.092 90)
+    (property "Value" "10k" (id 1) (at 217.17 99.9236 90))
+    (property "Footprint" "My_Misc:R_Axial_DIN0207_L6.3mm_D2.5mm_P10.16mm_Horizontal_larger_pads" (id 2) (at 217.17 101.092 90)
       (effects (font (size 1.27 1.27)) hide)
     )
@@
     (in_bom yes) (on_board yes)
     (property "Reference" "R7" (id 0) (at 217.17 107.7722 90))
-    (property "Value" "" (id 1) (at 217.17 110.0836 90))
-    (property "Footprint" "" (id 2) (at 217.17 111.252 90)
+    (property "Value" "10k" (id 1) (at 217.17 110.0836 90))
+    (property "Footprint" "My_Misc:R_Axial_DIN0207_L6.3mm_D2.5mm_P10.16mm_Horizontal_larger_pads" (id 2) (at 217.17 111.252 90)
       (effects (font (size 1.27 1.27)) hide)
     )
@@
     (in_bom yes) (on_board yes)
     (property "Reference" "R8" (id 0) (at 217.17 117.9322 90))
-    (property "Value" "" (id 1) (at 217.17 120.2436 90))
-    (property "Footprint" "" (id 2) (at 217.17 121.412 90)
+    (property "Value" "10k" (id 1) (at 217.17 120.2436 90))
+    (property "Footprint" "My_Misc:R_Axial_DIN0207_L6.3mm_D2.5mm_P10.16mm_Horizontal_larger_pads" (id 2) (at 217.17 121.412 90)
       (effects (font (size 1.27 1.27)) hide)
     )
@@
     )
     (path "/00000000-0000-0000-0000-00005e67312d"
-      (reference "J4") (unit 1) (value "3-pin_KY-019_relay_header") (footprint "My_Headers:3-pin JST KY-019 relay")
+      (reference "J4") (unit 1) (value "Bell relay") (footprint "My_Headers:3-pin JST KY-019 relay")
     )
     (path "/00000000-0000-0000-0000-00005e67ad35"
